Commit message: added wheels

File: description/robot_core.xacro (robot description, xacro)
@@ -19,5 +19,5 @@
  <link name="base_link"></link>
 <!-- Chassis link -->
-<joint name="chassis_name" type="fixed">
+<joint name="chassis_joint" type="fixed">
     <parent link="base_link"/>
     <child link="chassis"/>
@@ -45,3 +45,47 @@
     </inertial> -->
 </link>
+<!-- LEFT WHEEL LINK -->
+<joint name="left_wheel_joint" type="continuous">
+    <parent link="base_link" />
+    <child link="left_wheel" />
+    <origin xyz="0 0.175 0" rpy="-${pi/2} 0 0" />
+    <axis xyz=" 0 0 1" />
+</joint>
+<link name="left_wheel">
+    <visual>
+        <geometry>
+            <cylinder radius="0.05" length="0.04" />
+        </geometry>
+        <material name="blue" />
+    </visual>
+</link>
+<!-- RIGHT WHEEL LINK -->
+<joint name="right_wheel_joint" type="continuous">
+    <parent link="base_link" />
+    <child link="right_wheel" />
+    <origin xyz="0 -0.175 0" rpy="${pi/2} 0 0" />
+    <axis xyz=" 0 0 -1" />
+</joint>
+<link name="right_wheel">
+    <visual>
+        <geometry>
+            <cylinder radius="0.05" length="0.04" />
+        </geometry>
+        <material name="blue" />
+    </visual>
+</link>
+<!-- CASTER WHEEL LINK -->
+<joint name="caster_wheel_joint" type="fixed">
+    <parent link="chassis"/>
+    <child link="caster_wheel"/>
+    <origin xyz="0.24 0 0" />
+</joint>
+<link name="caster_wheel">
+    <visual>
+        <geometry>
+            <sphere radius="0.05" />
+        </geometry>
+        <material name="black" />
+    </visual>
+</link>
 </robot>

Commit message: added inertial xacro

File: description/robot_core.xacro (robot description, xacro)
@@ -1,4 +1,5 @@
 <?xml version="1.0"?>
 <robot xmlns:xacro="http://www.ros.org/wiki/xacro"  >
+<xacro:include filename="inertial_macros.xacro" />
 <material name="white">
     <color rgba=" 1 1 1 1"/>
@@ -26,5 +27,5 @@
 <link name="chassis">
     <visual>
-         <origin xyz="0.15 0 0.075" />
+        <origin xyz="0.15 0 0.075" />
         <geometry>
             <box size="0.3 0.3 0.15" />
@@ -32,16 +33,14 @@
         <material name="white" />
     </visual>
-    <!-- <collision>
+    <collision>
+        <origin xyz="0.15 0 0.075" />
         <geometry>
-            <mesh filename="package://pkg_name/meshes/file_name"/>
-            <box size="1.0 1.0 1.0" />
-            <cylinder radius="1.0" length="1.0"/>
+            <box size="0.3 0.3 0.15" />
         </geometry>
+        <material name="white" />
     </collision>
-    <inertial>
-        <mass value="0.0"/>
-        <origin xyz="0.0 0.0 0.0" rpy="0.0 0.0 0.0"/>
-        <inertia ixx="0.0" ixy="0.0" ixz="0.0" iyy="0.0" iyz="0.0" izz="0.0"/>
-    </inertial> -->
+    <xacro:inertial_box mass="0.5" x="0.5" y="0.3" z="0.15">
+        <origin xyz="0.15 0 0.075" rpy="0 0 0" />
+    </xacro:inertial_box>
 </link>
 <!-- LEFT WHEEL LINK -->
@@ -59,4 +58,13 @@
         <material name="blue" />
     </visual>
+    <collision>
+        <geometry>
+            <cylinder radius="0.05" length="0.04" />
+        </geometry>
+        <material name="blue" />
+    </collision>
+    <xacro:inertial_cylinder mass="0.1" length="0.44" radius="0.05" >
+        <origin xyz="0 0 0" rpy="0 0 0"/>
+    </xacro:inertial_cylinder>
 </link>
 <!-- RIGHT WHEEL LINK -->
@@ -74,4 +82,13 @@
         <material name="blue" />
     </visual>
+    <collision>
+        <geometry>
+            <cylinder radius="0.05" length="0.04" />
+        </geometry>
+        <material name="blue" />
+    </collision>
+    <xacro:inertial_cylinder mass="0.1" length="0.44" radius="0.05" >
+        <origin xyz="0 0 0" rpy="0 0 0"/>
+    </xacro:inertial_cylinder>
 </link>
 <!-- CASTER WHEEL LINK -->
@@ -88,4 +105,13 @@
         <material name="black" />
     </visual>
+    <collision>
+        <geometry>
+            <sphere radius="0.05" />
+        </geometry>
+        <material name="black" />
+    </collision>
+    <xacro:inertial_sphere mass="0.1" radius="0.05">
+        <origin xyz="0 0 0" rpy="0 0 0"/>
+    </xacro:inertial_sphere>
 </link>
 </robot>
