Commit message: added gazebo controls plugin

File: description/robot.urdf.xacro (robot description, xacro)
@@ -2,3 +2,4 @@
 <robot xmlns:xacro="http://www.ros.org/wiki/xacro"  name="robot">
     <xacro:include filename="robot_core.xacro"/>
+    <xacro:include filename="gazebo_control.xacro" />
 </robot>

File: description/robot_core.xacro (robot description, xacro)
@@ -44,4 +44,7 @@
     </xacro:inertial_box>
 </link>
+<gazebo reference="chassis">
+    <material>Gazebo/White</material>
+</gazebo>
 <!-- LEFT WHEEL LINK -->
 <joint name="left_wheel_joint" type="continuous">
@@ -68,4 +71,7 @@
     </xacro:inertial_cylinder>
 </link>
+<gazebo reference="left_wheel">
+    <material>Gazebo/Blue</material>
+</gazebo>
 <!-- RIGHT WHEEL LINK -->
 <joint name="right_wheel_joint" type="continuous">
@@ -92,4 +98,7 @@
     </xacro:inertial_cylinder>
 </link>
+<gazebo reference="right_wheel">
+    <material>Gazebo/Blue</material>
+</gazebo>
 <!-- CASTER WHEEL LINK -->
 <joint name="caster_wheel_joint" type="fixed">
@@ -115,3 +124,8 @@
     </xacro:inertial_sphere>
 </link>
+<gazebo reference="caster_wheel">
+    <material>Gazebo/Black</material>
+     <mu1 value="0.001"/>
+        <mu2 value="0.001"/>
+</gazebo>
 </robot>

Commit message: added lidar sensior in gazebo

File: description/robot.urdf.xacro (robot description, xacro)
@@ -3,3 +3,4 @@
     <xacro:include filename="robot_core.xacro"/>
     <xacro:include filename="gazebo_control.xacro" />
+    <xacro:include filename="lidar.xacro" />
 </robot>

File: description/robot_core.xacro (robot description, xacro)
@@ -16,4 +16,7 @@
 <material name="green">
     <color rgba=" 0 1 0 1"/>
+</material>
+<material name="red">
+    <color rgba=" 1 0 0 1"/>
 </material>
 <!-- Base link -->
